Commit message: URDF updated with remaining link comments

File: bringup/robot_description/urdf/4wheelrobot.xacro (robot description, xacro)
@@ -70,5 +70,5 @@
     <parent link="base_link"/>
     <child link="front_left_wheel"/>
-    <origin xyz="0.06 0.05 0"/>
+    <origin xyz="0.06 0.06 0"/>
   </joint>
   <!-- Front Right Wheel -->
@@ -85,5 +85,5 @@
     <parent link="base_link"/>
     <child link="front_right_wheel"/>
-    <origin xyz="0.06 -0.05 0"/>
+    <origin xyz="0.06 -0.06 0"/>
   </joint>
     <!-- Back Left Wheel-->
@@ -100,5 +100,5 @@
     <parent link="base_link"/>
     <child link="back_left_wheel"/>
-    <origin xyz="-0.06 0.05 0"/>
+    <origin xyz="-0.06 0.06 0"/>
   </joint>
   <!-- Back Right Wheel-->
@@ -115,5 +115,13 @@
     <parent link="base_link"/>
     <child link="back_right_wheel"/>
-    <origin xyz="-0.06 -0.05 0"/>
+    <origin xyz="-0.06 -0.06 0"/>
   </joint>
+  <!-- Distance sensor Left-->
+  <!-- Distance sensor Right-->
+  <!-- Linear actuator of type "continuous"-->
+  <!-- Rotary camera actuator of type "continuous"-->
+  <!-- Lidar above on base_link-->
+  <!-- nav_link of type "continuous"-->
+  <!-- IMU link on base_link-->
+  <!-- GPS link on base_link-->
 </robot>

Commit message: Dev: All URDF links (distance senor, imu, gps etc) added

File: bringup/robot_description/urdf/4wheelrobot.xacro (robot description, xacro)
@@ -118,10 +118,72 @@
   </joint>
   <!-- Distance sensor Left-->
+  <link name="left_distance_sensor">
+  </link>
+  <joint name="base_to_left_distance_sensor" type="fixed">
+    <parent link="base_link"/>
+    <child link="left_distance_sensor"/>
+    <origin xyz="0.1 0.02 0" rpy="0 0 0.3"/>
+    <!-- <origin rpy="1.57 1.57 -1.57"/> -->
+  </joint>
   <!-- Distance sensor Right-->
+  <link name="right_distance_sensor">
+  </link>
+  <joint name="base_to_right_distance_sensor" type="fixed">
+    <parent link="base_link"/>
+    <child link="right_distance_sensor"/>
+    <origin xyz="0.1 -0.02 0" rpy="0 0 -0.3"/>
+  </joint>
   <!-- Linear actuator of type "continuous"-->
-  <!-- Rotary camera actuator of type "continuous"-->
+  <link name="linear_link">
+  </link>
+  <joint name="base_to_linear_link" type="continuous">
+    <parent link="base_link"/>
+    <child link="linear_link"/>
+  </joint>
+  <!-- Rotary actuator of type "continuous"-->
+  <link name="rotary_link">
+  </link>
+  <joint name="linear_to_rotary_link" type="fixed">
+    <parent link="linear_link"/>
+    <child link="rotary_link"/>
+    <origin xyz="0 0.15 0"/>
+  </joint>
+    <!-- Camera actuator of type "continuous"-->
+  <link name="camera_link">
+  </link>
+  <joint name="rotary_to_camera_link" type="continuous">
+    <parent link="rotary_link"/>
+    <child link="camera_link"/>
+  </joint>
   <!-- Lidar above on base_link-->
+  <link name="lidar">
+  </link>
+  <joint name="base_to_lidar" type="fixed">
+    <parent link="base_link"/>
+    <child link="lidar"/>
+    <origin xyz="0 0 0.06"/>
+  </joint>
   <!-- nav_link of type "continuous"-->
+  <link name="nav_link">
+  </link>
+  <joint name="base_to_nav_link" type="continuous">
+    <parent link="base_link"/>
+    <child link="nav_link"/>
+  </joint>
   <!-- IMU link on base_link-->
+  <link name="imu">
+  </link>
+  <joint name="base_to_imu" type="fixed">
+    <parent link="base_link"/>
+    <child link="imu"/>
+    <origin xyz="0 0 0"/>
+  </joint>
   <!-- GPS link on base_link-->
+  <link name="gps">
+  </link>
+  <joint name="base_to_gps" type="fixed">
+    <parent link="base_link"/>
+    <child link="gps"/>
+    <origin xyz="0 0 0"/>
+  </joint>
 </robot>

Commit message: Updated urdf

File: bringup/robot_description/urdf/4wheelrobot.xacro (robot description, xacro)
@@ -1,42 +1,18 @@
 <?xml version="1.0"?>
-<robot
-    xmlns:gazebo="http://playerstage.sourceforge.net/gazebo/xmlschema/#gz"
-    xmlns:model="http://playerstage.sourceforge.net/gazebo/xmlschema/#model"
-    xmlns:sensor="http://playerstage.sourceforge.net/gazebo/xmlschema/#sensor"
-    xmlns:body="http://playerstage.sourceforge.net/gazebo/xmlschema/#body"
-    xmlns:geom="http://playerstage.sourceforge.net/gazebo/xmlschema/#geom"
-    xmlns:joint="http://playerstage.sourceforge.net/gazebo/xmlschema/#joint"
-    xmlns:controller="http://playerstage.sourceforge.net/gazebo/xmlschema/#controller"
-    xmlns:interface="http://playerstage.sourceforge.net/gazebo/xmlschema/#interface"
-    xmlns:rendering="http://playerstage.sourceforge.net/gazebo/xmlschema/#rendering"
-    xmlns:physics="http://playerstage.sourceforge.net/gazebo/xmlschema/#physics"
-    xmlns:xacro="http://www.ros.org/wiki/xacro" name="4wheelrobot">
-   <!-- Physical Material Macros -->
-    <material name="Red">
-    	<color rgba="1.0 0 0 1.0"/>
-    </material>
-    <material name="Green">
-    	<color rgba="0 1.0 0 1.0"/>
-    </material>
-    <material name="Blue">
-    	<color rgba="0 0 1.0 0.5"/>
-    </material>
-    <material name="Black">
-    	<color rgba="0 0 0 1.0"/>
-    </material>
-    <material name="Aqua">
-    	<color rgba="0 1.0 1.0 1.0"/>
-    </material>
-    <material name="black">
-      <color rgba="0.2 0.2 0.2 1."/>
-    </material>
-    <material name="blue">
-      <color rgba="0.3 0.57 1. 1."/>
-    </material>
-  <xacro:property name="wheelbase" value="0.1" />
+<robot xmlns:xacro="http://www.ros.org/wiki/xacro" name="4wheelrobot">
+  <!-- Color Macros -->
+  <material name="red">
+    <color rgba="1.0 0 0 1.0"/>
+  </material>
+  <material name="blue">
+    <color rgba="0.3 0.57 1. 1."/>
+  </material>
+  <!-- Base Properties -->
   <xacro:property name="body_length" value="0.2" />
   <xacro:property name="body_width" value="0.1" />
   <xacro:property name="body_height" value="0.05" />
   <xacro:property name="ground_offset" value="0.04" />
+  <!-- Wheel Properties -->
+  <xacro:property name="wheelbase" value="0.1" />
   <xacro:property name="wheel_radius" value="0.04" />
   <xacro:property name="wheel_length" value="0.02" />
